Commit message: add imu sensor

File: delivery_description/urdf/delivery.urdf.xacro (robot description, xacro)
@@ -270,3 +270,33 @@
       friction="0.1" />
   </joint>
+  <link name="imu_link">
+    <inertial>
+      <origin xyz="-0.00552433659106688 0.000168210391520346 0.000514000497342681" rpy="0 0 0" />
+      <mass value="0.000528415362211671" />
+      <inertia ixx="1.46176048428261E-08" ixy="1.40015117949421E-10" ixz="-1.99633872937403E-12"
+               iyy="8.59662482954888E-09" iyz="7.52375112767959E-12"
+               izz="2.30279421279312E-08" />
+    </inertial>
+    <visual>
+      <origin xyz="0 0 0" rpy="0 0 0" />
+      <geometry>
+        <mesh filename="package://delivery_description/meshes/imu_link.STL" />
+      </geometry>
+      <material name="">
+        <color rgba="0.792156862745098 0.819607843137255 0.933333333333333 1" />
+      </material>
+    </visual>
+    <collision>
+      <origin xyz="0 0 0" rpy="0 0 0" />
+      <geometry>
+        <mesh filename="package://delivery_description/meshes/imu_link.STL" />
+      </geometry>
+    </collision>
+  </link>
+  <joint name="imu_joint" type="fixed">
+    <origin xyz="0 0 0" rpy="0 0 0" />
+    <parent link="base_link" />
+    <child link="imu_link" />
+    <axis xyz="0 0 0" />
+  </joint>
 </robot>

File: delivery_description/urdf/delivery_gazebo.xacro (robot description, xacro)
@@ -83,4 +83,6 @@
         <parameters>$(find delivery_controller)/config/delivery_controllers.yaml</parameters>
       </plugin>
+      <plugin filename="ignition-gazebo-imu-system" name="ignition::gazebo::systems::Imu">
+      </plugin>
     </xacro:if>
     <!-- ROS 2 Iron or above -->
@@ -89,5 +91,58 @@
         <parameters>$(find delivery_controller)/config/delivery_controllers.yaml</parameters>
       </plugin>
+      <plugin filename="gz-sim-imu-system" name="gz::sim::systems::Imu">
+      </plugin>
     </xacro:unless>
+  </gazebo>
+  <!-- IMU -->
+  <gazebo reference="imu_link">
+    <sensor name="imu" type="imu">
+        <always_on>true</always_on>
+        <update_rate>100</update_rate>
+        <gz_frame_id>imu_link</gz_frame_id>
+        <topic>imu</topic>
+        <imu>
+          <angular_velocity>
+            <x>
+              <noise type="gaussian">
+                <mean>0.0</mean>
+                <stddev>2e-4</stddev>
+              </noise>
+            </x>
+            <y>
+              <noise type="gaussian">
+                <mean>0.0</mean>
+                <stddev>2e-4</stddev>
+              </noise>
+            </y>
+            <z>
+              <noise type="gaussian">
+                <mean>0.0</mean>
+                <stddev>2e-4</stddev>
+              </noise>
+            </z>
+          </angular_velocity>
+          <linear_acceleration>
+            <x>
+              <noise type="gaussian">
+                <mean>0.0</mean>
+                <stddev>1.7e-2</stddev>
+              </noise>
+            </x>
+            <y>
+              <noise type="gaussian">
+                <mean>0.0</mean>
+                <stddev>1.7e-2</stddev>
+              </noise>
+            </y>
+            <z>
+              <noise type="gaussian">
+                <mean>0.0</mean>
+                <stddev>1.7e-2</stddev>
+              </noise>
+            </z>
+          </linear_acceleration>
+        </imu>
+    </sensor>
   </gazebo>
   <!-- <gazebo>

Commit message: add 2D Laser Scanner

File: delivery_description/urdf/delivery.urdf.xacro (robot description, xacro)
@@ -300,3 +300,43 @@
     <axis xyz="0 0 0" />
   </joint>
+    <link name="laser_link">
+    <inertial>
+      <origin xyz="-0.011945780406062 -0.000381929217680526 -0.0170649378129477" rpy="0 0 0" />
+      <mass value="0.073084435549317" />
+      <inertia ixx="1.96074931730795E-05" ixy="-3.62091076640009E-07" ixz="4.28230084046735E-07"
+               iyy="2.40983835136327E-05" iyz="1.50180909250652E-08"
+               izz="4.14184164228595E-05" />
+    </inertial>
+    <visual>
+      <origin xyz="0 0 0" rpy="0 0 0" />
+      <geometry>
+        <mesh filename="package://delivery_description/meshes/laser_link.STL" />
+      </geometry>
+      <material name="dark_grey"/>
+    </visual>
+    <collision>
+      <origin xyz="0 0 0" rpy="0 0 0" />
+      <geometry>
+        <mesh filename="package://delivery_description/meshes/laser_link.STL" />
+      </geometry>
+    </collision>
+  </link>
+  <joint name="laser_joint" type="fixed">
+    <origin xyz="0.2 0 0.035" rpy="0 0 0" />
+    <parent link="base_link" />
+    <child link="laser_link" />
+    <axis xyz="0 0 0" />
+  </joint>
+  <material name="blue">
+    <color rgba="0 0 1 1"/>
+  </material>
+  <material name="black">
+    <color rgba="0 0 0 1"/>
+  </material>
+  <material name="silver">
+    <color rgba="0.79 0.82 0.93 1"/>
+  </material>
+  <material name="dark_grey">
+    <color rgba="0.3 0.3 0.3 1"/>
+  </material>
 </robot>

File: delivery_description/urdf/delivery_gazebo.xacro (robot description, xacro)
@@ -85,4 +85,7 @@
       <plugin filename="ignition-gazebo-imu-system" name="ignition::gazebo::systems::Imu">
       </plugin>
+      <plugin filename="ignition-gazebo-sensors-system" name="ignition::gazebo::systems::Sensors">
+        <render_engine>ogre2</render_engine>
+      </plugin>
     </xacro:if>
     <!-- ROS 2 Iron or above -->
@@ -92,4 +95,7 @@
       </plugin>
       <plugin filename="gz-sim-imu-system" name="gz::sim::systems::Imu">
+      </plugin>
+      <plugin filename="gz-sim-sensors-system" name="gz::sim::systems::Sensors">
+        <render_engine>ogre2</render_engine>
       </plugin>
     </xacro:unless>
@@ -144,4 +150,34 @@
           </linear_acceleration>
         </imu>
+    </sensor>
+  </gazebo>
+   <!-- 2D Laser Sensor -->
+  <gazebo reference="laser_link">
+    <sensor name="lidar" type="gpu_lidar">
+      <always_on>true</always_on>
+      <visualize>true</visualize>
+      <topic>scan</topic>
+      <update_rate>5</update_rate>
+      <gz_frame_id>laser_link</gz_frame_id>
+      <lidar>
+        <scan>
+          <horizontal>
+            <samples>360</samples>
+            <resolution>1.00000</resolution>
+            <min_angle>0.000000</min_angle>
+            <max_angle>6.280000</max_angle>
+          </horizontal>
+        </scan>
+        <range>
+          <min>0.120000</min>
+          <max>12.0</max>
+          <resolution>0.02</resolution>
+        </range>
+        <noise>
+          <type>gaussian</type>
+          <mean>0.0</mean>
+          <stddev>0.01</stddev>
+        </noise>
+      </lidar>
     </sensor>
   </gazebo>

Commit message: add Camera

File: delivery_description/urdf/delivery.urdf.xacro (robot description, xacro)
@@ -30,9 +30,5 @@
         <mesh filename="package://delivery_description/meshes/base_link.STL" />
       </geometry>
-      <material
-        name="">
-        <color
-          rgba="0.1 0.1 0.1 1" />
-      </material>
+      <material name="black" />
     </visual>
     <collision>
@@ -328,4 +324,30 @@
     <axis xyz="0 0 0" />
   </joint>
+  <link name="camera_link">
+        <visual>
+            <geometry>
+                <box size="0.01 0.1 0.05" />
+            </geometry>
+            <material name="silver" />
+        </visual>
+        <collision>
+            <geometry>
+                <box size="0.01 0.1 0.05" />
+            </geometry>
+        </collision>
+        <!-- <xacro:box_inertia m="0.1" x="0.01" y="0.1" z="0.05"
+                           o_xyz="0 0 0" o_rpy="0 0 0" /> -->
+  </link>
+  <joint name="base_camera_joint" type="fixed">
+        <parent link="base_link" />
+        <child link="camera_link" />
+        <origin xyz="0.25 0 -0.05" rpy="0 0 0" />
+    </joint>
+  <link name="camera_link_optical" />
+  <joint name="camera_optical_joint" type="fixed">
+        <origin xyz="0 0 0" rpy="${-pi/2} 0 ${-pi/2}"/>
+        <parent link="camera_link"/>
+        <child link="camera_link_optical"/>
+  </joint>
   <material name="blue">
     <color rgba="0 0 1 1"/>

File: delivery_description/urdf/delivery_gazebo.xacro (robot description, xacro)
@@ -182,4 +182,31 @@
     </sensor>
   </gazebo>
+  <gazebo reference="camera_link">
+        <sensor name="camera" type="camera">
+            <camera>
+                <horizontal_fov>1.3962634</horizontal_fov>
+                <image>
+                    <width>640</width>
+                    <height>480</height>
+                    <format>R8G8B8</format>
+                </image>
+                <clip>
+                    <near>0.1</near>
+                    <far>15</far>
+                </clip>
+                <noise>
+                    <type>gaussian</type>
+                    <mean>0.0</mean>
+                    <stddev>0.007</stddev>
+                </noise>
+                <optical_frame_id>camera_link_optical</optical_frame_id>
+                <camera_info_topic>camera/camera_info</camera_info_topic>
+            </camera>
+            <always_on>1</always_on>
+            <update_rate>20</update_rate>
+            <visualize>true</visualize>
+            <topic>camera/image_raw</topic>
+        </sensor>
+    </gazebo>
   <!-- <gazebo>
     <xacro:if value="$(arg is_ignition)">

Commit message: Tuning friction(mu,mu2) for mecanum wheels

File: delivery_description/urdf/delivery.urdf.xacro (robot description, xacro)
@@ -76,8 +76,8 @@
     <collision>
       <origin
-        xyz="0 0.03 0"
-        rpy="1.5708 0 0" />
-      <geometry>
-        <mesh filename="package://delivery_description/meshes/Front_Left_Wheel.STL" />
+        xyz="0 0 0"
+        rpy="1.5708 0 0" />
+      <geometry>
+        <cylinder radius="0.05" length="0.058" />
       </geometry>
     </collision>
@@ -131,8 +131,8 @@
     <collision>
       <origin
-        xyz="0 -0.03 0"
-        rpy="1.5708 0 0" />
-      <geometry>
-        <mesh filename="package://delivery_description/meshes/Right_Front_Wheel.STL" />
+        xyz="0 0 0"
+        rpy="1.5708 0 0" />
+      <geometry>
+        <cylinder radius="0.05" length="0.058" />
       </geometry>
     </collision>
@@ -186,8 +186,8 @@
     <collision>
       <origin
-        xyz="0 0.03 0"
-        rpy="1.5708 0 0" />
-      <geometry>
-        <mesh filename="package://delivery_description/meshes/Left_Back_wheel.STL" />
+        xyz="0 0 0"
+        rpy="1.5708 0 0" />
+      <geometry>
+        <cylinder radius="0.05" length="0.058" />
       </geometry>
     </collision>
@@ -241,8 +241,8 @@
     <collision>
       <origin
-        xyz="0 -0.03 0"
-        rpy="1.5708 0 0" />
-      <geometry>
-        <mesh filename="package://delivery_description/meshes/Right_Bach_Wheel.STL" />
+        xyz="0 0 0"
+        rpy="1.5708 0 0" />
+      <geometry>
+        <cylinder radius="0.05" length="0.058" />
       </geometry>
     </collision>

File: delivery_description/urdf/delivery_gazebo.xacro (robot description, xacro)
@@ -3,54 +3,70 @@
   <!-- Wheels -->
   <gazebo reference="front_left_wheel">
-    <collision>
-      <surface>
-        <friction>
-          <ode>
-            <mu>1.0</mu>
-            <mu2>0.8</mu2>
-            <fdir1 gz:expressed_in="base_link">1 1 0</fdir1>
-          </ode>
-        </friction>
-      </surface>
-    </collision>
+     <collision>
+          <surface>
+            <friction>
+              <ode>
+                <mu>1.5</mu>
+                <mu2>0.7</mu2>
+                <kp>200000.0</kp>
+                <kd>5000.0</kd>
+                <slip1>0.035</slip1>
+                <slip2>0</slip2>
+                <fdir1 gz:expressed_in="base_footprint">1 -1 0</fdir1>
+              </ode>
+            </friction>
+          </surface>
+        </collision>
   </gazebo>
   <gazebo reference="front_right_wheel">
     <collision>
-      <surface>
-        <friction>
-          <ode>
-            <mu>1.0</mu>
-            <mu2>0.8</mu2>
-            <fdir1 gz:expressed_in="base_link">1 -1 0</fdir1>
-          </ode>
-        </friction>
-      </surface>
-    </collision>
+          <surface>
+            <friction>
+              <ode>
+                <mu>1.5</mu>
+                <mu2>0.7</mu2>
+                <kp>200000.0</kp>
+                <kd>5000.0</kd>
+                <slip1>0.035</slip1>
+                <slip2>0</slip2>
+                <fdir1 gz:expressed_in="base_footprint">1 1 0</fdir1>
+              </ode>
+            </friction>
+          </surface>
+        </collision>
   </gazebo>
   <gazebo reference="back_left_wheel">
     <collision>
-      <surface>
-        <friction>
-          <ode>
-            <mu>1.0</mu>
-            <mu2>0.8</mu2>
-            <fdir1 gz:expressed_in="base_link">-1 1 0</fdir1>
-          </ode>
-        </friction>
-      </surface>
-    </collision>
+          <surface>
+            <friction>
+              <ode>
+                <mu>1.5</mu>
+                <mu2>0.7</mu2>
+                <kp>200000.0</kp>
+                <kd>5000.0</kd>
+                <slip1>0.035</slip1>
+                <slip2>0</slip2>
+                <fdir1 gz:expressed_in="base_footprint">1 1 0</fdir1>
+              </ode>
+            </friction>
+          </surface>
+        </collision>
   </gazebo>
   <gazebo reference="back_right_wheel">
     <collision>
-      <surface>
-        <friction>
-          <ode>
-            <mu>1.0</mu>
-            <mu2>0.8</mu2>
-            <fdir1 gz:expressed_in="base_link">-1 -1 0</fdir1>
-          </ode>
-        </friction>
-      </surface>
-    </collision>
+          <surface>
+            <friction>
+              <ode>
+                <mu>1.5</mu>
+                <mu2>0.7</mu2>
+                <kp>200000.0</kp>
+                <kd>5000.0</kd>
+                <slip1>0.035</slip1>
+                <slip2>0</slip2>
+                <fdir1 gz:expressed_in="base_footprint">1 -1 0</fdir1>
+              </ode>
+            </friction>
+          </surface>
+        </collision>
   </gazebo>
   <gazebo>

Commit message: add pose publisher plugin to gazebo

File: delivery_description/urdf/delivery.urdf.xacro (robot description, xacro)
@@ -12,5 +12,5 @@
   <link name="base_link">
     <inertial>
-      <origin xyz="0 0 -0.05" rpy="0 0 0" />
+      <origin xyz="0 0 0" rpy="0 0 0" />
       <mass
         value="50" />
@@ -25,5 +25,5 @@
     <visual>
       <origin
-        xyz="0 0 0"
+        xyz="0 0 0.1"
         rpy="0 0 0" />
       <geometry>
@@ -34,5 +34,5 @@
     <collision>
       <origin
-        xyz="0 0 0"
+        xyz="0 0 0.1"
         rpy="0 0 0" />
       <geometry>
@@ -44,5 +44,5 @@
       <parent link="base_footprint" />
       <child link="base_link" />
-      <origin xyz="0 0 0.21" rpy="0 0 0"/>
+      <origin xyz="0 0 0.11" rpy="0 0 0"/>
   </joint>
   <link name="front_left_wheel">
@@ -86,5 +86,5 @@
     type="continuous">
     <origin
-      xyz="0.19721 0.24498 -0.15567"
+      xyz="0.19721 0.24498 -0.05567"
       rpy="0 0 0" />
     <parent
@@ -141,5 +141,5 @@
     type="continuous">
     <origin
-      xyz="0.19721 -0.24502 -0.15567"
+      xyz="0.19721 -0.24502 -0.05567"
       rpy="0 0 0" />
     <parent
@@ -196,5 +196,5 @@
     type="continuous">
     <origin
-      xyz="-0.19721 0.24498 -0.15567"
+      xyz="-0.19721 0.24498 -0.05567"
       rpy="0 0 0" />
     <parent
@@ -251,5 +251,5 @@
     type="continuous">
     <origin
-      xyz="-0.19721 -0.24502 -0.15567"
+      xyz="-0.19721 -0.24502 -0.05567"
       rpy="0 0 0" />
     <parent
@@ -319,5 +319,5 @@
   </link>
   <joint name="laser_joint" type="fixed">
-    <origin xyz="0.2 0 0.035" rpy="0 0 0" />
+    <origin xyz="0.2 0 0.135" rpy="0 0 0" />
     <parent link="base_link" />
     <child link="laser_link" />
@@ -342,5 +342,5 @@
         <parent link="base_link" />
         <child link="camera_link" />
-        <origin xyz="0.25 0 -0.05" rpy="0 0 0" />
+        <origin xyz="0.25 0 0.05" rpy="0 0 0" />
     </joint>
   <link name="camera_link_optical" />

File: delivery_description/urdf/delivery_gazebo.xacro (robot description, xacro)
@@ -115,4 +115,18 @@
         <render_engine>ogre2</render_engine>
       </plugin>
+      <plugin
+        filename="gz-sim-pose-publisher-system"
+        name="gz::sim::systems::PosePublisher">
+        <!-- We don’t need link, visual, collision, or sensor-specific poses -->
+        <publish_link_pose>false</publish_link_pose>
+        <publish_visual_pose>false</publish_visual_pose>
+        <publish_collision_pose>false</publish_collision_pose>
+        <publish_sensor_pose>false</publish_sensor_pose>
+        <!-- Publish a single pose instead of a Pose_V list -->
+        <use_pose_vector_msg>false</use_pose_vector_msg>
+        <!-- These two options ensure the robot model pose is published -->
+        <publish_model_pose>true</publish_model_pose>
+        <publish_nested_model_pose>true</publish_nested_model_pose>
+    </plugin>
     </xacro:unless>
   </gazebo>

Commit message: change wheel collision to sphere

File: delivery_description/urdf/delivery.urdf.xacro (robot description, xacro)
@@ -79,5 +79,5 @@
         rpy="1.5708 0 0" />
       <geometry>
-        <cylinder radius="0.05" length="0.058" />
+        <sphere radius="0.05" />
       </geometry>
     </collision>
@@ -134,5 +134,5 @@
         rpy="1.5708 0 0" />
       <geometry>
-        <cylinder radius="0.05" length="0.058" />
+        <sphere radius="0.05" />
       </geometry>
     </collision>
@@ -189,5 +189,5 @@
         rpy="1.5708 0 0" />
       <geometry>
-        <cylinder radius="0.05" length="0.058" />
+        <sphere radius="0.05" />
       </geometry>
     </collision>
@@ -244,5 +244,5 @@
         rpy="1.5708 0 0" />
       <geometry>
-        <cylinder radius="0.05" length="0.058" />
+        <sphere radius="0.05" />
       </geometry>
     </collision>
@@ -294,5 +294,4 @@
     <parent link="base_link" />
     <child link="imu_link" />
-    <axis xyz="0 0 0" />
   </joint>
     <link name="laser_link">
@@ -322,5 +321,4 @@
     <parent link="base_link" />
     <child link="laser_link" />
-    <axis xyz="0 0 0" />
   </joint>
   <link name="camera_link">
