Commit message: modifid urdf

File: delivery_description/urdf/delivery.urdf.xacro (robot description, xacro)
@@ -1,6 +1,3 @@
 <?xml version="1.0"?>
-<!-- This URDF was automatically created by SolidWorks to URDF Exporter! Originally created by Stephen Brawner (brawner@gmail.com)
-     Commit Version: 1.6.0-4-g7f85cfe  Build Version: 1.6.7995.38578
-     For more information, please see http://wiki.ros.org/sw_urdf_exporter -->
 <robot name="delivery" xmlns:xacro="http://ros.org/wiki/xacro">
   <xacro:arg name="is_ignition" default="true" />
@@ -18,8 +15,8 @@
       <inertia
         ixx="0.190013298612022"
-        ixy="-1.97362982292358E-06"
-        ixz="1.09139279405602E-15"
+        ixy="0"
+        ixz="0"
         iyy="0.194102599343596"
-        iyz="-1.36853189937296E-17"
+        iyz="0"
         izz="0.328271696632787" />
     </inertial>
@@ -56,8 +53,8 @@
       <inertia
         ixx="8.05457942683617E-05"
-        ixy="-2.79543633711077E-15"
-        ixz="3.37021382345757E-14"
+        ixy="0"
+        ixz="0"
         iyy="8.05457942749361E-05"
-        iyz="1.10037676592356E-14"
+        iyz="0"
         izz="9.3195603890608E-05" />
     </inertial>
@@ -98,7 +95,7 @@
       effort="180"
       velocity="50" />
-    <dynamics
+    <!-- <dynamics
       damping="0.1"
-      friction="0.1" />
+      friction="0.1" /> -->
   </joint>
   <link name="front_right_wheel">
@@ -110,10 +107,10 @@
         value="0.266614983222909" />
       <inertia
-        ixx="8.0545794268312E-05"
-        ixy="-2.80019667850405E-15"
-        ixz="3.37091076216657E-14"
-        iyy="8.05457942748739E-05"
-        iyz="1.10097155984234E-14"
-        izz="9.31956038905408E-05" />
+        ixx="8.05457942683617E-05"
+        ixy="0"
+        ixz="0"
+        iyy="8.05457942749361E-05"
+        iyz="0"
+        izz="9.3195603890608E-05" />
     </inertial>
     <visual>
@@ -153,7 +150,7 @@
       effort="180"
       velocity="50" />
-    <dynamics
+    <!-- <dynamics
       damping="0.1"
-      friction="0.1" />
+      friction="0.1" /> -->
   </joint>
   <link name="back_left_wheel">
@@ -165,10 +162,10 @@
         value="0.266614983222911" />
       <inertia
-        ixx="8.05457942683817E-05"
-        ixy="-2.79572074526522E-15"
-        ixz="3.36987949955329E-14"
-        iyy="8.05457942749372E-05"
-        iyz="1.10377338930185E-14"
-        izz="9.31956038906202E-05" />
+        ixx="8.05457942683617E-05"
+        ixy="0"
+        ixz="0"
+        iyy="8.05457942749361E-05"
+        iyz="0"
+        izz="9.3195603890608E-05" />
     </inertial>
     <visual>
@@ -208,7 +205,7 @@
       effort="180"
       velocity="50" />
-    <dynamics
+    <!-- <dynamics
       damping="0.1"
-      friction="0.1" />
+      friction="0.1" /> -->
   </joint>
   <link name="back_right_wheel">
@@ -220,10 +217,10 @@
         value="0.266614983222911" />
       <inertia
-        ixx="8.05457942683914E-05"
-        ixy="-2.79608823622019E-15"
-        ixz="3.36986637054261E-14"
-        iyy="8.05457942749527E-05"
-        iyz="1.10332704558511E-14"
-        izz="9.31956038906356E-05" />
+        ixx="8.05457942683617E-05"
+        ixy="0"
+        ixz="0"
+        iyy="8.05457942749361E-05"
+        iyz="0"
+        izz="9.3195603890608E-05" />
     </inertial>
     <visual>
@@ -263,7 +260,7 @@
       effort="180"
       velocity="50" />
-    <dynamics
+    <!-- <dynamics
       damping="0.1"
-      friction="0.1" />
+      friction="0.1" /> -->
   </joint>
   <link name="imu_link">

File: delivery_description/urdf/delivery_gazebo.xacro (robot description, xacro)
@@ -5,5 +5,4 @@
     <collision>
       <surface>
-        <!-- Contact dynamics -->
         <contact>
           <ode>
@@ -15,9 +14,9 @@
         <friction>
           <ode>
-            <mu>1.1</mu>
-            <mu2>0.07</mu2>
-            <slip1>0.015</slip1>
-            <slip2>0.14</slip2>
-            <fdir1 gz:expressed_in="base_footprint">1 1 0</fdir1>
+            <mu>0.6</mu>
+            <mu2>0.14</mu2>
+            <!-- <slip1>0.015</slip1> -->
+            <!-- <slip2>0.14</slip2> -->
+            <fdir1 gz:expressed_in="base_footprint">1 -1 0</fdir1>
           </ode>
         </friction>
@@ -38,9 +37,9 @@
         <friction>
           <ode>
-            <mu>1.1</mu>
-            <mu2>0.07</mu2>
-            <slip1>0.015</slip1>
-            <slip2>0.14</slip2>
-            <fdir1 gz:expressed_in="base_footprint">1 -1 0</fdir1>
+            <mu>0.6</mu>
+            <mu2>0.14</mu2>
+            <!-- <slip1>0.015</slip1> -->
+            <!-- <slip2>0.14</slip2> -->
+            <fdir1 gz:expressed_in="base_footprint">1 1 0</fdir1>
           </ode>
         </friction>
@@ -61,9 +60,9 @@
         <friction>
           <ode>
-            <mu>1.1</mu>
-            <mu2>0.07</mu2>
-            <slip1>0.015</slip1>
-            <slip2>0.14</slip2>
-            <fdir1 gz:expressed_in="base_footprint">1 -1 0</fdir1>
+            <mu>0.6</mu>
+            <mu2>0.14</mu2>
+            <!-- <slip1>0.015</slip1> -->
+            <!-- <slip2>0.14</slip2> -->
+            <fdir1 gz:expressed_in="base_footprint">1 1 0</fdir1>
           </ode>
         </friction>
@@ -84,9 +83,9 @@
         <friction>
           <ode>
-            <mu>1.1</mu>
-            <mu2>0.07</mu2>
-            <slip1>0.015</slip1>
-            <slip2>0.14</slip2>
-            <fdir1 gz:expressed_in="base_footprint">1 1 0</fdir1>
+            <mu>0.6</mu>
+            <mu2>0.14</mu2>
+            <!-- <slip1>0.015</slip1> -->
+            <!-- <slip2>0.14</slip2> -->
+            <fdir1 gz:expressed_in="base_footprint">1 -1 0</fdir1>
           </ode>
         </friction>
@@ -159,5 +158,5 @@
     <sensor name="imu" type="imu">
         <always_on>true</always_on>
-        <update_rate>100</update_rate>
+        <update_rate>15.0</update_rate>
         <gz_frame_id>imu_link</gz_frame_id>
         <topic>imu</topic>
@@ -212,5 +211,5 @@
       <visualize>true</visualize>
       <topic>scan</topic>
-      <update_rate>5</update_rate>
+      <update_rate>5.0</update_rate>
       <gz_frame_id>laser_link</gz_frame_id>
       <lidar>
@@ -228,9 +227,9 @@
           <resolution>0.02</resolution>
         </range>
-        <noise>
+        <!-- <noise>
           <type>gaussian</type>
           <mean>0.0</mean>
           <stddev>0.01</stddev>
-        </noise>
+        </noise> -->
       </lidar>
     </sensor>
@@ -258,5 +257,5 @@
             </camera>
             <always_on>1</always_on>
-            <update_rate>20</update_rate>
+            <update_rate>5.0</update_rate>
             <visualize>true</visualize>
             <topic>camera/image_raw</topic>
@@ -287,4 +286,9 @@
           <back_left_joint>back_left_wheel_joint</back_left_joint>
           <back_right_joint>back_right_wheel_joint</back_right_joint>
+          <odom_topic>mecanum_controller/odom</odom_topic>
+          <odom_frame_id>odom</odom_frame_id>
+          <frame_id>odom</frame_id>
+          <enable_odom_tf>true</enable_odom_tf>
+          <child_frame_id>base_footprint</child_frame_id>
           <wheel_separation>0.55</wheel_separation>
           <wheelbase>0.39442</wheelbase>
