Commit message: first commit

File: delivery_description/urdf/delivery_mobile_base.xacro (robot description, xacro)
@@ -10,5 +10,5 @@
   <xacro:include filename="$(find delivery_description)/urdf/delivery_gazebo.xacro"/>
   <!-- ROS2 Control-->
-  <xacro:include filename="$(find delivery_description)/urdf/delivery_ros2_control.xacro"/>
+  <!-- <xacro:include filename="$(find delivery_description)/urdf/delivery_ros2_control.xacro"/> -->
   <link name="base_footprint" />
   <link name="base_link">
@@ -280,3 +280,214 @@
     <color rgba="0.3 0.3 0.3 1"/>
   </material>
+  <!-- arm -->
+    <material name="grey">
+        <color rgba="0.5 0.5 0.5 1" />
+    </material>
+    <material name="dark_green">
+        <color rgba="0 0.4 0 1" />
+    </material>
+    <material name="light_green">
+        <color rgba="0 0.6 0 1" />
+    </material>
+    <link name="arm_base">
+        <visual>
+            <geometry>
+                <box size="0.098 0.098 0.005" />
+            </geometry>
+            <origin xyz="0 0 0.0025" rpy="0 0 0" />
+            <material name="grey" />
+        </visual>
+        <collision>
+            <geometry>
+                <box size="0.098 0.098 0.005" />
+            </geometry>
+            <origin xyz="0 0 0.0025" rpy="0 0 0" />
+        </collision>
+    </link>
+    <link name="shoulder_link">
+        <visual>
+            <geometry>
+                <cylinder length="0.04601" radius="0.044" />
+            </geometry>
+            <origin xyz="0 0 0.023005" rpy="0 0 0" />
+            <material name="blue" />
+        </visual>
+        <collision>
+            <geometry>
+                <cylinder length="0.04601" radius="0.044" />
+            </geometry>
+            <origin xyz="0 0 0.023005" rpy="0 0 0" />
+        </collision>
+    </link>
+    <link name="arm_link">
+        <visual>
+            <geometry>
+                <cylinder length="0.11312" radius="0.013" />
+            </geometry>
+            <origin xyz="0 0 0.05656" rpy="0 0 0" />
+            <material name="grey" />
+        </visual>
+        <collision>
+            <geometry>
+                <box size="0.026 0.026 0.11312" />
+            </geometry>
+            <origin xyz="0 0 0.05656" rpy="0 0 0" />
+        </collision>
+    </link>
+    <link name="elbow_link">
+        <visual>
+            <geometry>
+                <cylinder length="0.09795" radius="0.010885" />
+            </geometry>
+            <origin xyz="0 0 0.048975" rpy="0 0 0" />
+            <material name="blue" />
+        </visual>
+        <collision>
+            <geometry>
+                <box size="0.02177 0.02177 0.09795" />
+            </geometry>
+            <origin xyz="0 0 0.048975" rpy="0 0 0" />
+        </collision>
+    </link>
+    <link name="forearm_link">
+        <visual>
+            <geometry>
+                <box size="0.013 0.013 0.02908" />
+            </geometry>
+            <origin xyz="0 0 0.01454" rpy="0 0 0" />
+            <material name="grey" />
+        </visual>
+        <collision>
+            <geometry>
+                <box size="0.013 0.013 0.02908" />
+            </geometry>
+            <origin xyz="0 0 0.01454" rpy="0 0 0" />
+        </collision>
+    </link>
+    <link name="wrist_link">
+        <visual>
+            <geometry>
+                <box size="0.02177 0.02177 0.01999" />
+            </geometry>
+            <origin xyz="0 0 0.009995" rpy="0 0 0" />
+            <material name="blue" />
+        </visual>
+        <collision>
+            <geometry>
+                <box size="0.02177 0.02177 0.01099" />
+            </geometry>
+            <origin xyz="0 0 0.009995" rpy="0 0 0" />
+        </collision>
+    </link>
+    <link name="tool_link" />
+      <joint name="arm_base_joint" type="fixed">
+        <parent link="base_link" />
+        <child link="arm_base" />
+        <origin xyz="-0.2 0 0.1" rpy="0 0 0" />
+    </joint>
+    <joint name="joint1" type="revolute">
+        <parent link="arm_base" />
+        <child link="shoulder_link" />
+        <origin xyz="0 0 0.005" rpy="0 0 0" />
+        <axis xyz="0 0 1" />
+        <limit effort="1000.0" velocity="1.0" lower="-1.57" upper="1.57" />
+    </joint>
+    <joint name="joint2" type="revolute">
+        <parent link="shoulder_link" />
+        <child link="arm_link" />
+        <origin xyz="0 0 0.04601" rpy="0 0 0" />
+        <axis xyz="0 1 0" />
+        <limit effort="1000.0" velocity="1.0" lower="-1.57" upper="1.57" />
+    </joint>
+    <joint name="joint3" type="revolute">
+        <parent link="arm_link" />
+        <child link="elbow_link" />
+        <origin xyz="0 0 0.11312" rpy="0 0 0" />
+        <axis xyz="0 1 0" />
+        <limit effort="1000.0" velocity="1.0" lower="-1.57" upper="1.57" />
+    </joint>
+    <joint name="joint4" type="revolute">
+        <parent link="elbow_link" />
+        <child link="forearm_link" />
+        <origin xyz="0 0 0.09795" rpy="0 0 0" />
+        <axis xyz="0 0 1" />
+        <limit effort="1000.0" velocity="1.0" lower="-1.57" upper="1.57" />
+    </joint>
+    <joint name="joint5" type="revolute">
+        <parent link="forearm_link" />
+        <child link="wrist_link" />
+        <origin xyz="0 0 0.02908" rpy="0 0 0" />
+        <axis xyz="0 1 0" />
+        <limit effort="1000.0" velocity="1.0" lower="-1.57" upper="1.57" />
+    </joint>
+    <joint name="hand_tool_joint" type="fixed">
+        <parent link="wrist_link" />
+        <child link="tool_link" />
+        <origin xyz="0 0 0.009995" rpy="0 0 0" />
+    </joint>
+    <link name="gripper_base_link">
+        <visual>
+            <geometry>
+                <box size="0.1 0.03 0.02" />
+            </geometry>
+            <origin xyz="0 0 0.01" rpy="0 0 1.57" />
+            <material name="dark_green" />
+        </visual>
+        <collision>
+            <geometry>
+                <box size="0.1 0.03 0.02" />
+            </geometry>
+            <origin xyz="0 0 0.01" rpy="0 0 1.57" />
+        </collision>
+    </link>
+    <link name="gripper_left_finger_link">
+        <visual>
+            <geometry>
+                <box size="0.01 0.03 0.04" />
+            </geometry>
+            <origin xyz="0 0 0.02" rpy="0 0 1.57" />
+            <material name="light_green" />
+        </visual>
+        <collision>
+            <geometry>
+                <box size="0.01 0.03 0.04" />
+            </geometry>
+            <origin xyz="0 0 0.02" rpy="0 0 1.57" />
+        </collision>
+    </link>
+    <link name="gripper_right_finger_link">
+        <visual>
+            <geometry>
+                <box size="0.01 0.03 0.04" />
+            </geometry>
+            <origin xyz="0 0 0.02" rpy="0 0 1.57" />
+            <material name="light_green" />
+        </visual>
+        <collision>
+            <geometry>
+                <box size="0.01 0.03 0.04" />
+            </geometry>
+            <origin xyz="0 0 0.02" rpy="0 0 1.57" />
+        </collision>
+    </link>
+    <joint name="gripper_left_finger_joint" type="prismatic">
+        <parent link="gripper_base_link" />
+        <child link="gripper_left_finger_link" />
+        <origin xyz="0 -0.04 0.02" rpy="0 0 0" />
+        <axis xyz="0 1 0" />
+        <limit effort="1000.0" velocity="1.0" lower="0.0" upper="0.035" />
+    </joint>
+    <joint name="gripper_right_finger_joint" type="prismatic">
+        <parent link="gripper_base_link" />
+        <child link="gripper_right_finger_link" />
+        <origin xyz="0 0.04 0.02" rpy="0 0 0" />
+        <axis xyz="0 1 0" />
+        <mimic joint="gripper_left_finger_joint" multiplier="-1.0" />
+        <limit effort="1000.0" velocity="1.0" lower="-0.035" upper="0.0" />
+    </joint>
+    <joint name="gripper_base_joint" type="fixed">
+        <parent link="tool_link" />
+        <child link="gripper_base_link" />
+        <origin xyz="0 0 0" rpy="0 0 0" />
+    </joint>
 </robot>

Commit message: fixing robot arm and scan topic

File: delivery_description/urdf/delivery_mobile_base.xacro (robot description, xacro)
@@ -280,3 +280,313 @@
     <color rgba="0.3 0.3 0.3 1"/>
   </material>
+  <!-- arm -->
+    <material name="grey">
+        <color rgba="0.5 0.5 0.5 1" />
+    </material>
+    <material name="dark_green">
+        <color rgba="0 0.4 0 1" />
+    </material>
+    <material name="light_green">
+        <color rgba="0 0.6 0 1" />
+    </material>
+    <link name="arm_base">
+        <inertial>
+            <origin xyz="0 0 0.0025" rpy="0 0 0" />
+            <mass value="0.05" />
+            <inertia
+                ixx="4.012E-05"
+                ixy="0"
+                ixz="0"
+                iyy="4.012E-05"
+                iyz="0"
+                izz="8.003E-05" />
+        </inertial>
+        <visual>
+            <geometry>
+                <box size="0.098 0.098 0.005" />
+            </geometry>
+            <origin xyz="0 0 0.0025" rpy="0 0 0" />
+            <material name="grey" />
+        </visual>
+        <collision>
+            <geometry>
+                <box size="0.098 0.098 0.005" />
+            </geometry>
+            <origin xyz="0 0 0.0025" rpy="0 0 0" />
+        </collision>
+    </link>
+    <link name="shoulder_link">
+        <inertial>
+            <origin xyz="0 0 0.023005" rpy="0 0 0" />
+            <mass value="0.15" />
+            <inertia
+                ixx="9.906E-05"
+                ixy="0"
+                ixz="0"
+                iyy="9.906E-05"
+                iyz="0"
+                izz="1.452E-04" />
+        </inertial>
+        <visual>
+            <geometry>
+                <cylinder length="0.04601" radius="0.044" />
+            </geometry>
+            <origin xyz="0 0 0.023005" rpy="0 0 0" />
+            <material name="blue" />
+        </visual>
+        <collision>
+            <geometry>
+                <cylinder length="0.04601" radius="0.044" />
+            </geometry>
+            <origin xyz="0 0 0.023005" rpy="0 0 0" />
+        </collision>
+    </link>
+    <link name="arm_link">
+        <inertial>
+            <origin xyz="0 0 0.05656" rpy="0 0 0" />
+            <mass value="0.05" />
+            <inertia
+                ixx="5.518E-05"
+                ixy="0"
+                ixz="0"
+                iyy="5.518E-05"
+                iyz="0"
+                izz="4.225E-06" />
+        </inertial>
+        <visual>
+            <geometry>
+                <cylinder length="0.11312" radius="0.013" />
+            </geometry>
+            <origin xyz="0 0 0.05656" rpy="0 0 0" />
+            <material name="grey" />
+        </visual>
+        <collision>
+            <geometry>
+                <box size="0.026 0.026 0.11312" />
+            </geometry>
+            <origin xyz="0 0 0.05656" rpy="0 0 0" />
+        </collision>
+    </link>
+    <link name="elbow_link">
+        <inertial>
+            <origin xyz="0 0 0.048975" rpy="0 0 0" />
+            <mass value="0.03" />
+            <inertia
+                ixx="2.501E-05"
+                ixy="0"
+                ixz="0"
+                iyy="2.501E-05"
+                iyz="0"
+                izz="1.777E-06" />
+        </inertial>
+        <visual>
+            <geometry>
+                <cylinder length="0.09795" radius="0.010885" />
+            </geometry>
+            <origin xyz="0 0 0.048975" rpy="0 0 0" />
+            <material name="blue" />
+        </visual>
+        <collision>
+            <geometry>
+                <box size="0.02177 0.02177 0.09795" />
+            </geometry>
+            <origin xyz="0 0 0.048975" rpy="0 0 0" />
+        </collision>
+    </link>
+    <link name="forearm_link">
+        <inertial>
+            <origin xyz="0 0 0.01454" rpy="0 0 0" />
+            <mass value="0.01" />
+            <inertia
+                ixx="8.297E-07"
+                ixy="0"
+                ixz="0"
+                iyy="8.297E-07"
+                iyz="0"
+                izz="2.817E-07" />
+        </inertial>
+        <visual>
+            <geometry>
+                <box size="0.013 0.013 0.02908" />
+            </geometry>
+            <origin xyz="0 0 0.01454" rpy="0 0 0" />
+            <material name="grey" />
+        </visual>
+        <collision>
+            <geometry>
+                <box size="0.013 0.013 0.02908" />
+            </geometry>
+            <origin xyz="0 0 0.01454" rpy="0 0 0" />
+        </collision>
+    </link>
+    <link name="wrist_link">
+        <inertial>
+            <origin xyz="0 0 0.009995" rpy="0 0 0" />
+            <mass value="0.01" />
+            <inertia
+                ixx="7.279E-07"
+                ixy="0"
+                ixz="0"
+                iyy="7.279E-07"
+                iyz="0"
+                izz="7.898E-07" />
+        </inertial>
+        <visual>
+            <geometry>
+                <box size="0.02177 0.02177 0.01999" />
+            </geometry>
+            <origin xyz="0 0 0.009995" rpy="0 0 0" />
+            <material name="blue" />
+        </visual>
+        <collision>
+            <geometry>
+                <box size="0.02177 0.02177 0.01099" />
+            </geometry>
+            <origin xyz="0 0 0.009995" rpy="0 0 0" />
+        </collision>
+    </link>
+    <link name="tool_link" />
+      <joint name="arm_base_joint" type="fixed">
+        <parent link="base_link" />
+        <child link="arm_base" />
+        <origin xyz="-0.2 0 0.1" rpy="0 0 0" />
+    </joint>
+    <joint name="joint1" type="revolute">
+        <parent link="arm_base" />
+        <child link="shoulder_link" />
+        <origin xyz="0 0 0.005" rpy="0 0 0" />
+        <axis xyz="0 0 1" />
+        <limit effort="1000.0" velocity="1.0" lower="-1.57" upper="1.57" />
+    </joint>
+    <joint name="joint2" type="revolute">
+        <parent link="shoulder_link" />
+        <child link="arm_link" />
+        <origin xyz="0 0 0.04601" rpy="0 0 0" />
+        <axis xyz="0 1 0" />
+        <limit effort="1000.0" velocity="1.0" lower="-1.57" upper="1.57" />
+    </joint>
+    <joint name="joint3" type="revolute">
+        <parent link="arm_link" />
+        <child link="elbow_link" />
+        <origin xyz="0 0 0.11312" rpy="0 0 0" />
+        <axis xyz="0 1 0" />
+        <limit effort="1000.0" velocity="1.0" lower="-1.57" upper="1.57" />
+    </joint>
+    <joint name="joint4" type="revolute">
+        <parent link="elbow_link" />
+        <child link="forearm_link" />
+        <origin xyz="0 0 0.09795" rpy="0 0 0" />
+        <axis xyz="0 0 1" />
+        <limit effort="1000.0" velocity="1.0" lower="-1.57" upper="1.57" />
+    </joint>
+    <joint name="joint5" type="revolute">
+        <parent link="forearm_link" />
+        <child link="wrist_link" />
+        <origin xyz="0 0 0.02908" rpy="0 0 0" />
+        <axis xyz="0 1 0" />
+        <limit effort="1000.0" velocity="1.0" lower="-1.57" upper="1.57" />
+    </joint>
+    <joint name="hand_tool_joint" type="fixed">
+        <parent link="wrist_link" />
+        <child link="tool_link" />
+        <origin xyz="0 0 0.009995" rpy="0 0 0" />
+    </joint>
+    <link name="gripper_base_link">
+        <inertial>
+            <origin xyz="0 0 0.01" rpy="0 0 1.57" />
+            <mass value="0.05" />
+            <inertia
+                ixx="5.417E-06"
+                ixy="0"
+                ixz="0"
+                iyy="4.333E-05"
+                iyz="0"
+                izz="4.542E-05" />
+        </inertial>
+        <visual>
+            <geometry>
+                <box size="0.1 0.03 0.02" />
+            </geometry>
+            <origin xyz="0 0 0.01" rpy="0 0 1.57" />
+            <material name="dark_green" />
+        </visual>
+        <collision>
+            <geometry>
+                <box size="0.1 0.03 0.02" />
+            </geometry>
+            <origin xyz="0 0 0.01" rpy="0 0 1.57" />
+        </collision>
+    </link>
+    <link name="gripper_left_finger_link">
+        <inertial>
+            <origin xyz="0 0 0.02" rpy="0 0 1.57" />
+            <mass value="0.01" />
+            <inertia
+                ixx="2.083E-06"
+                ixy="0"
+                ixz="0"
+                iyy="1.417E-06"
+                iyz="0"
+                izz="8.333E-07" />
+        </inertial>
+        <visual>
+            <geometry>
+                <box size="0.01 0.03 0.04" />
+            </geometry>
+            <origin xyz="0 0 0.02" rpy="0 0 1.57" />
+            <material name="light_green" />
+        </visual>
+        <collision>
+            <geometry>
+                <box size="0.01 0.03 0.04" />
+            </geometry>
+            <origin xyz="0 0 0.02" rpy="0 0 1.57" />
+        </collision>
+    </link>
+    <link name="gripper_right_finger_link">
+        <inertial>
+            <origin xyz="0 0 0.02" rpy="0 0 1.57" />
+            <mass value="0.01" />
+            <inertia
+                ixx="2.083E-06"
+                ixy="0"
+                ixz="0"
+                iyy="1.417E-06"
+                iyz="0"
+                izz="8.333E-07" />
+        </inertial>
+        <visual>
+            <geometry>
+                <box size="0.01 0.03 0.04" />
+            </geometry>
+            <origin xyz="0 0 0.02" rpy="0 0 1.57" />
+            <material name="light_green" />
+        </visual>
+        <collision>
+            <geometry>
+                <box size="0.01 0.03 0.04" />
+            </geometry>
+            <origin xyz="0 0 0.02" rpy="0 0 1.57" />
+        </collision>
+    </link>
+    <joint name="gripper_left_finger_joint" type="prismatic">
+        <parent link="gripper_base_link" />
+        <child link="gripper_left_finger_link" />
+        <origin xyz="0 -0.04 0.02" rpy="0 0 0" />
+        <axis xyz="0 1 0" />
+        <limit effort="1000.0" velocity="1.0" lower="0.0" upper="0.035" />
+    </joint>
+    <joint name="gripper_right_finger_joint" type="prismatic">
+        <parent link="gripper_base_link" />
+        <child link="gripper_right_finger_link" />
+        <origin xyz="0 0.04 0.02" rpy="0 0 0" />
+        <axis xyz="0 1 0" />
+        <mimic joint="gripper_left_finger_joint" multiplier="-1.0" />
+        <limit effort="1000.0" velocity="1.0" lower="-0.035" upper="0.0" />
+    </joint>
+    <joint name="gripper_base_joint" type="fixed">
+        <parent link="tool_link" />
+        <child link="gripper_base_link" />
+        <origin xyz="0 0 0" rpy="0 0 0" />
+    </joint>
 </robot>

File: delivery_description/urdf/delivery_ros2_control.xacro (robot description, xacro)
@@ -11,5 +11,5 @@
             </joint>
     </xacro:macro>
-    <ros2_control name="MobileSystem" type="system">
+    <ros2_control name="Mobile_System" type="system">
         <!-- ros2_control Gazebo -->
         <xacro:if value="$(arg is_sim)">
@@ -40,3 +40,70 @@
         <xacro:wheel_control side="back_right" />
     </ros2_control>
+    <ros2_control name="Maniplutor_System" type="system">
+        <!-- ros2_control Gazebo -->
+        <xacro:if value="$(arg is_sim)">
+            <!-- ROS 2 Humble -->
+            <xacro:if value="$(arg is_ignition)">
+                <hardware>
+                    <plugin>ign_ros2_control/IgnitionSystem</plugin>
+                </hardware>
+            </xacro:if>
+            <!-- ROS 2 Iron or above -->
+            <xacro:unless value="$(arg is_ignition)">
+                <hardware>
+                    <plugin>gz_ros2_control/GazeboSimSystem</plugin>
+                </hardware>
+            </xacro:unless>
+        </xacro:if>
+        <!-- ros2_control Real Robot -->
+        <xacro:unless value="$(arg is_sim)">
+            <hardware>
+                <plugin>delivery_firmware/DeliveryFirmware</plugin>
+                <param name="device">/dev/ttyUSB0</param>
+                <param name="baud_rate">115200</param>
+            </hardware>
+        </xacro:unless>
+        <joint name="joint1">
+            <command_interface name="position"/>
+            <state_interface name="position">
+                <param name="initial_value">0</param>
+            </state_interface>
+            <state_interface name="velocity"/>
+        </joint>
+        <joint name="joint2">
+            <command_interface name="position"/>
+            <state_interface name="position">
+                <param name="initial_value">0</param>
+            </state_interface>
+            <state_interface name="velocity"/>
+        </joint>
+        <joint name="joint3">
+            <command_interface name="position"/>
+            <state_interface name="position">
+                <param name="initial_value">0</param>
+            </state_interface>
+            <state_interface name="velocity"/>
+        </joint>
+        <joint name="joint4">
+            <command_interface name="position"/>
+            <state_interface name="position">
+                <param name="initial_value">0</param>
+            </state_interface>
+            <state_interface name="velocity"/>
+        </joint>
+        <joint name="joint5">
+            <command_interface name="position"/>
+            <state_interface name="position">
+                <param name="initial_value">0</param>
+            </state_interface>
+            <state_interface name="velocity"/>
+        </joint>
+        <joint name="gripper_left_finger_joint">
+            <command_interface name="position"/>
+            <state_interface name="position">
+                <param name="initial_value">0</param>
+            </state_interface>
+            <state_interface name="velocity"/>
+        </joint>
+    </ros2_control>
 </robot>
