Commit message: #

File: delivery_description/urdf/delivery_gazebo.xacro (robot description, xacro)
@@ -1,40 +1,56 @@
 <?xml version="1.0" ?>
-<robot name="delivery"  xmlns:xacro="http://ros.org/wiki/xacro">
+<robot name="delivery"  xmlns:xacro="http://ros.org/wiki/xacro" xmlns:gz="http://gazebosim.org/schema">
   <!-- Wheels -->
   <gazebo reference="front_left_wheel">
-    <mu1>1e15</mu1>
-    <mu2>1e13</mu2>
-    <kp>1e10</kp>
-    <kd>1000.0</kd>
-    <minDepth>0.001</minDepth>
-    <maxVel>0.5</maxVel>
-    <fdir1>1 1 0</fdir1>
+    <collision>
+      <surface>
+        <friction>
+          <ode>
+            <mu>1.0</mu>
+            <mu2>0.8</mu2>
+            <fdir1 gz:expressed_in="base_link">1 1 0</fdir1>
+          </ode>
+        </friction>
+      </surface>
+    </collision>
   </gazebo>
   <gazebo reference="front_right_wheel">
-    <mu1>1e15</mu1>
-    <mu2>1e13</mu2>
-    <kp>1e10</kp>
-    <kd>1000.0</kd>
-    <minDepth>0.001</minDepth>
-    <maxVel>0.5</maxVel>
-    <fdir1>-1 1 0</fdir1>
+    <collision>
+      <surface>
+        <friction>
+          <ode>
+            <mu>1.0</mu>
+            <mu2>0.8</mu2>
+            <fdir1 gz:expressed_in="base_link">1 -1 0</fdir1>
+          </ode>
+        </friction>
+      </surface>
+    </collision>
   </gazebo>
   <gazebo reference="back_left_wheel">
-    <mu1>1e15</mu1>
-    <mu2>1e13</mu2>
-    <kp>1e10</kp>
-    <kd>1000.0</kd>
-    <minDepth>0.001</minDepth>
-    <maxVel>0.5</maxVel>
-    <fdir1>-1 -1 0</fdir1>
+    <collision>
+      <surface>
+        <friction>
+          <ode>
+            <mu>1.0</mu>
+            <mu2>0.8</mu2>
+            <fdir1 gz:expressed_in="base_link">-1 1 0</fdir1>
+          </ode>
+        </friction>
+      </surface>
+    </collision>
   </gazebo>
   <gazebo reference="back_right_wheel">
-    <mu1>1e15</mu1>
-    <mu2>1e13</mu2>
-    <kp>1e10</kp>
-    <kd>1000.0</kd>
-    <minDepth>0.001</minDepth>
-    <maxVel>0.5</maxVel>
-    <fdir1>1 -1 0</fdir1>
+    <collision>
+      <surface>
+        <friction>
+          <ode>
+            <mu>1.0</mu>
+            <mu2>0.8</mu2>
+            <fdir1 gz:expressed_in="base_link">-1 -1 0</fdir1>
+          </ode>
+        </friction>
+      </surface>
+    </collision>
   </gazebo>
   <gazebo>
@@ -75,3 +91,35 @@
     </xacro:unless>
   </gazebo>
+  <!-- <gazebo>
+    <xacro:if value="$(arg is_ignition)">
+      <plugin
+          filename="ign-sim-mecanum-drive-system"
+          name="libign::sim::systems::MecanumDrive">
+          <front_left_joint>front_left_wheel_joint</front_left_joint>
+          <front_right_joint>front_right_wheel_joint</front_right_joint>
+          <back_left_joint>back_left_wheel_joint</back_left_joint>
+          <back_right_joint>back_right_wheel_joint</back_right_joint>
+          <wheel_separation>0.55</wheel_separation>
+          <wheelbase>0.39442</wheelbase>
+          <wheel_radius>0.05</wheel_radius>
+          <min_acceleration>-5</min_acceleration>
+          <max_acceleration>5</max_acceleration>
+        </plugin>
+      </xacro:if>
+    <xacro:unless value="$(arg is_ignition)">
+      <plugin
+          filename="gz-sim-mecanum-drive-system"
+          name="gz::sim::systems::MecanumDrive">
+          <front_left_joint>front_left_wheel_joint</front_left_joint>
+          <front_right_joint>front_right_wheel_joint</front_right_joint>
+          <back_left_joint>back_left_wheel_joint</back_left_joint>
+          <back_right_joint>back_right_wheel_joint</back_right_joint>
+          <wheel_separation>0.55</wheel_separation>
+          <wheelbase>0.39442</wheelbase>
+          <wheel_radius>0.05</wheel_radius>
+          <min_acceleration>-5</min_acceleration>
+          <max_acceleration>5</max_acceleration>
+        </plugin>
+    </xacro:unless>
+  </gazebo> -->
 </robot>

Commit message: update friction coefficient

File: delivery_description/urdf/delivery_gazebo.xacro (robot description, xacro)
@@ -3,72 +3,96 @@
   <!-- Wheels -->
   <gazebo reference="front_left_wheel">
-     <collision>
-          <surface>
-            <friction>
-              <ode>
-                <mu>1.5</mu>
-                <mu2>0.7</mu2>
-                <kp>200000.0</kp>
-                <kd>5000.0</kd>
-                <slip1>0.035</slip1>
-                <slip2>0</slip2>
-                <fdir1 gz:expressed_in="base_footprint">1 -1 0</fdir1>
-              </ode>
-            </friction>
-          </surface>
-        </collision>
+    <collision>
+      <surface>
+        <!-- Contact dynamics -->
+        <contact>
+          <ode>
+            <kp>1.5e6</kp>
+            <kd>2e4</kd>
+          </ode>
+        </contact>
+        <!-- Friction properties -->
+        <friction>
+          <ode>
+            <mu>1.1</mu>
+            <mu2>0.07</mu2>
+            <slip1>0.015</slip1>
+            <slip2>0.14</slip2>
+            <fdir1 gz:expressed_in="base_footprint">1 -1 0</fdir1>
+          </ode>
+        </friction>
+      </surface>
+    </collision>
   </gazebo>
   <gazebo reference="front_right_wheel">
     <collision>
-          <surface>
-            <friction>
-              <ode>
-                <mu>1.5</mu>
-                <mu2>0.7</mu2>
-                <kp>200000.0</kp>
-                <kd>5000.0</kd>
-                <slip1>0.035</slip1>
-                <slip2>0</slip2>
-                <fdir1 gz:expressed_in="base_footprint">1 1 0</fdir1>
-              </ode>
-            </friction>
-          </surface>
-        </collision>
+      <surface>
+        <!-- Contact dynamics -->
+        <contact>
+          <ode>
+            <kp>1.5e6</kp>
+            <kd>2e4</kd>
+          </ode>
+        </contact>
+        <!-- Friction properties -->
+        <friction>
+          <ode>
+            <mu>1.1</mu>
+            <mu2>0.07</mu2>
+            <slip1>0.015</slip1>
+            <slip2>0.14</slip2>
+            <fdir1 gz:expressed_in="base_footprint">1 1 0</fdir1>
+          </ode>
+        </friction>
+      </surface>
+    </collision>
   </gazebo>
   <gazebo reference="back_left_wheel">
     <collision>
-          <surface>
-            <friction>
-              <ode>
-                <mu>1.5</mu>
-                <mu2>0.7</mu2>
-                <kp>200000.0</kp>
-                <kd>5000.0</kd>
-                <slip1>0.035</slip1>
-                <slip2>0</slip2>
-                <fdir1 gz:expressed_in="base_footprint">1 1 0</fdir1>
-              </ode>
-            </friction>
-          </surface>
-        </collision>
+      <surface>
+        <!-- Contact dynamics -->
+        <contact>
+          <ode>
+            <kp>1.5e6</kp>
+            <kd>2e4</kd>
+          </ode>
+        </contact>
+        <!-- Friction properties -->
+        <friction>
+          <ode>
+            <mu>1.1</mu>
+            <mu2>0.07</mu2>
+            <slip1>0.015</slip1>
+            <slip2>0.14</slip2>
+            <fdir1 gz:expressed_in="base_footprint">1 1 0</fdir1>
+          </ode>
+        </friction>
+      </surface>
+    </collision>
   </gazebo>
   <gazebo reference="back_right_wheel">
     <collision>
-          <surface>
-            <friction>
-              <ode>
-                <mu>1.5</mu>
-                <mu2>0.7</mu2>
-                <kp>200000.0</kp>
-                <kd>5000.0</kd>
-                <slip1>0.035</slip1>
-                <slip2>0</slip2>
-                <fdir1 gz:expressed_in="base_footprint">1 -1 0</fdir1>
-              </ode>
-            </friction>
-          </surface>
-        </collision>
-  </gazebo>
-  <gazebo>
+      <surface>
+        <!-- Contact dynamics -->
+        <contact>
+          <ode>
+            <kp>1.5e6</kp>
+            <kd>2e4</kd>
+          </ode>
+        </contact>
+        <!-- Friction properties -->
+        <friction>
+          <ode>
+            <mu>1.1</mu>
+            <mu2>0.07</mu2>
+            <slip1>0.015</slip1>
+            <slip2>0.14</slip2>
+            <fdir1 gz:expressed_in="base_footprint">1 -1 0</fdir1>
+          </ode>
+        </friction>
+      </surface>
+    </collision>
+  </gazebo>
+  <!-- <gazebo>
     <xacro:if value="$(arg is_ignition)">
       <plugin
@@ -91,5 +115,5 @@
       </plugin>
     </xacro:unless>
-  </gazebo>
+  </gazebo> -->
   <!-- ROS 2 Control -->
   <gazebo>

Commit message: change friction direction for mecanum roller

File: delivery_description/urdf/delivery_gazebo.xacro (robot description, xacro)
@@ -19,4 +19,27 @@
             <slip1>0.015</slip1>
             <slip2>0.14</slip2>
+            <fdir1 gz:expressed_in="base_footprint">1 1 0</fdir1>
+          </ode>
+        </friction>
+      </surface>
+    </collision>
+  </gazebo>
+  <gazebo reference="front_right_wheel">
+    <collision>
+      <surface>
+        <!-- Contact dynamics -->
+        <contact>
+          <ode>
+            <kp>1.5e6</kp>
+            <kd>2e4</kd>
+          </ode>
+        </contact>
+        <!-- Friction properties -->
+        <friction>
+          <ode>
+            <mu>1.1</mu>
+            <mu2>0.07</mu2>
+            <slip1>0.015</slip1>
+            <slip2>0.14</slip2>
             <fdir1 gz:expressed_in="base_footprint">1 -1 0</fdir1>
           </ode>
@@ -25,5 +48,28 @@
     </collision>
   </gazebo>
-  <gazebo reference="front_right_wheel">
+  <gazebo reference="back_left_wheel">
+    <collision>
+      <surface>
+        <!-- Contact dynamics -->
+        <contact>
+          <ode>
+            <kp>1.5e6</kp>
+            <kd>2e4</kd>
+          </ode>
+        </contact>
+        <!-- Friction properties -->
+        <friction>
+          <ode>
+            <mu>1.1</mu>
+            <mu2>0.07</mu2>
+            <slip1>0.015</slip1>
+            <slip2>0.14</slip2>
+            <fdir1 gz:expressed_in="base_footprint">1 -1 0</fdir1>
+          </ode>
+        </friction>
+      </surface>
+    </collision>
+  </gazebo>
+  <gazebo reference="back_right_wheel">
     <collision>
       <surface>
@@ -43,50 +89,4 @@
             <slip2>0.14</slip2>
             <fdir1 gz:expressed_in="base_footprint">1 1 0</fdir1>
-          </ode>
-        </friction>
-      </surface>
-    </collision>
-  </gazebo>
-  <gazebo reference="back_left_wheel">
-    <collision>
-      <surface>
-        <!-- Contact dynamics -->
-        <contact>
-          <ode>
-            <kp>1.5e6</kp>
-            <kd>2e4</kd>
-          </ode>
-        </contact>
-        <!-- Friction properties -->
-        <friction>
-          <ode>
-            <mu>1.1</mu>
-            <mu2>0.07</mu2>
-            <slip1>0.015</slip1>
-            <slip2>0.14</slip2>
-            <fdir1 gz:expressed_in="base_footprint">1 1 0</fdir1>
-          </ode>
-        </friction>
-      </surface>
-    </collision>
-  </gazebo>
-  <gazebo reference="back_right_wheel">
-    <collision>
-      <surface>
-        <!-- Contact dynamics -->
-        <contact>
-          <ode>
-            <kp>1.5e6</kp>
-            <kd>2e4</kd>
-          </ode>
-        </contact>
-        <!-- Friction properties -->
-        <friction>
-          <ode>
-            <mu>1.1</mu>
-            <mu2>0.07</mu2>
-            <slip1>0.015</slip1>
-            <slip2>0.14</slip2>
-            <fdir1 gz:expressed_in="base_footprint">1 -1 0</fdir1>
           </ode>
         </friction>

Commit message: clean and minimze xacro file

File: delivery_description/urdf/delivery_gazebo.xacro (robot description, xacro)
@@ -1,5 +1,40 @@
 <?xml version="1.0" ?>
-<robot name="delivery"  xmlns:xacro="http://ros.org/wiki/xacro" xmlns:gz="http://gazebosim.org/schema">
+<robot  xmlns:xacro="http://ros.org/wiki/xacro" xmlns:gz="http://gazebosim.org/schema">
   <!-- Wheels -->
+  <xacro:macro name="wheel_collision" params="side">
+        <xacro:if value="${side == 'front_left'}">
+            <xacro:property name="fdir" value="1 -1 0" />
+        </xacro:if>
+        <xacro:if value="${side == 'back_right'}">
+            <xacro:property name="fdir" value="1 -1 0" />
+        </xacro:if>
+        <xacro:if value="${side == 'front_right'}">
+            <xacro:property name="fdir" value="1 1 0" />
+        </xacro:if>
+        <xacro:if value="${side == 'back_left'}">
+            <xacro:property name="fdir" value="1 1 0" />
+        </xacro:if>
+        <gazebo reference="${side}_wheel">
+            <collision>
+                <surface>
+                    <contact>
+                        <ode>
+                            <kp>1.5e6</kp>
+                            <kd>2e4</kd>
+                        </ode>
+                    </contact>
+                    <friction>
+                        <ode>
+                            <mu>0.6</mu>
+                            <mu2>0.14</mu2>
+                            <!-- <slip1>0.015</slip1> -->
+                            <!-- <slip2>0.14</slip2> -->
+                            <fdir1 gz:expressed_in="base_footprint">${fdir}</fdir1>
+                        </ode>
+                    </friction>
+                </surface>
+            </collision>
+        </gazebo>
+  </xacro:macro>
   <gazebo reference="front_left_wheel">
     <collision>
@@ -93,26 +128,4 @@
     </collision>
   </gazebo>
-  <!-- <gazebo>
-    <xacro:if value="$(arg is_ignition)">
-      <plugin
-          filename="ignition-joint-state-publisher-system"
-          name="ignition::systems::JointStatePublisher">
-          <joint_name>front_left_wheel_joint</joint_name>
-          <joint_name>front_right_wheel_joint</joint_name>
-          <joint_name>back_left_wheel_joint</joint_name>
-          <joint_name>back_right_wheel_joint</joint_name>
-      </plugin>
-    </xacro:if>
-    <xacro:unless value="$(arg is_ignition)">
-     <plugin
-        filename="gz-sim-joint-state-publisher-system"
-        name="gz::sim::systems::JointStatePublisher">
-          <joint_name>front_left_wheel_joint</joint_name>
-          <joint_name>front_right_wheel_joint</joint_name>
-          <joint_name>back_left_wheel_joint</joint_name>
-          <joint_name>back_right_wheel_joint</joint_name>
-      </plugin>
-    </xacro:unless>
-  </gazebo> -->
   <!-- ROS 2 Control -->
   <gazebo>
@@ -262,40 +275,3 @@
         </sensor>
     </gazebo>
-  <!-- <gazebo>
-    <xacro:if value="$(arg is_ignition)">
-      <plugin
-          filename="ign-sim-mecanum-drive-system"
-          name="libign::sim::systems::MecanumDrive">
-          <front_left_joint>front_left_wheel_joint</front_left_joint>
-          <front_right_joint>front_right_wheel_joint</front_right_joint>
-          <back_left_joint>back_left_wheel_joint</back_left_joint>
-          <back_right_joint>back_right_wheel_joint</back_right_joint>
-          <wheel_separation>0.55</wheel_separation>
-          <wheelbase>0.39442</wheelbase>
-          <wheel_radius>0.05</wheel_radius>
-          <min_acceleration>-5</min_acceleration>
-          <max_acceleration>5</max_acceleration>
-        </plugin>
-      </xacro:if>
-    <xacro:unless value="$(arg is_ignition)">
-      <plugin
-          filename="gz-sim-mecanum-drive-system"
-          name="gz::sim::systems::MecanumDrive">
-          <front_left_joint>front_left_wheel_joint</front_left_joint>
-          <front_right_joint>front_right_wheel_joint</front_right_joint>
-          <back_left_joint>back_left_wheel_joint</back_left_joint>
-          <back_right_joint>back_right_wheel_joint</back_right_joint>
-          <odom_topic>mecanum_controller/odom</odom_topic>
-          <odom_frame_id>odom</odom_frame_id>
-          <frame_id>odom</frame_id>
-          <enable_odom_tf>true</enable_odom_tf>
-          <child_frame_id>base_footprint</child_frame_id>
-          <wheel_separation>0.55</wheel_separation>
-          <wheelbase>0.39442</wheelbase>
-          <wheel_radius>0.05</wheel_radius>
-          <min_acceleration>-5</min_acceleration>
-          <max_acceleration>5</max_acceleration>
-        </plugin>
-    </xacro:unless>
-  </gazebo> -->
 </robot>

Commit message: clesn xacro

File: delivery_description/urdf/delivery_gazebo.xacro (robot description, xacro)
@@ -37,95 +37,8 @@
         </gazebo>
   </xacro:macro>
-  <gazebo reference="front_left_wheel">
-    <collision>
-      <surface>
-        <contact>
-          <ode>
-            <kp>1.5e6</kp>
-            <kd>2e4</kd>
-          </ode>
-        </contact>
-        <!-- Friction properties -->
-        <friction>
-          <ode>
-            <mu>0.6</mu>
-            <mu2>0.14</mu2>
-            <!-- <slip1>0.015</slip1> -->
-            <!-- <slip2>0.14</slip2> -->
-            <fdir1 gz:expressed_in="base_footprint">1 -1 0</fdir1>
-          </ode>
-        </friction>
-      </surface>
-    </collision>
-  </gazebo>
-  <gazebo reference="front_right_wheel">
-    <collision>
-      <surface>
-        <!-- Contact dynamics -->
-        <contact>
-          <ode>
-            <kp>1.5e6</kp>
-            <kd>2e4</kd>
-          </ode>
-        </contact>
-        <!-- Friction properties -->
-        <friction>
-          <ode>
-            <mu>0.6</mu>
-            <mu2>0.14</mu2>
-            <!-- <slip1>0.015</slip1> -->
-            <!-- <slip2>0.14</slip2> -->
-            <fdir1 gz:expressed_in="base_footprint">1 1 0</fdir1>
-          </ode>
-        </friction>
-      </surface>
-    </collision>
-  </gazebo>
-  <gazebo reference="back_left_wheel">
-    <collision>
-      <surface>
-        <!-- Contact dynamics -->
-        <contact>
-          <ode>
-            <kp>1.5e6</kp>
-            <kd>2e4</kd>
-          </ode>
-        </contact>
-        <!-- Friction properties -->
-        <friction>
-          <ode>
-            <mu>0.6</mu>
-            <mu2>0.14</mu2>
-            <!-- <slip1>0.015</slip1> -->
-            <!-- <slip2>0.14</slip2> -->
-            <fdir1 gz:expressed_in="base_footprint">1 1 0</fdir1>
-          </ode>
-        </friction>
-      </surface>
-    </collision>
-  </gazebo>
-  <gazebo reference="back_right_wheel">
-    <collision>
-      <surface>
-        <!-- Contact dynamics -->
-        <contact>
-          <ode>
-            <kp>1.5e6</kp>
-            <kd>2e4</kd>
-          </ode>
-        </contact>
-        <!-- Friction properties -->
-        <friction>
-          <ode>
-            <mu>0.6</mu>
-            <mu2>0.14</mu2>
-            <!-- <slip1>0.015</slip1> -->
-            <!-- <slip2>0.14</slip2> -->
-            <fdir1 gz:expressed_in="base_footprint">1 -1 0</fdir1>
-          </ode>
-        </friction>
-      </surface>
-    </collision>
-  </gazebo>
+  <xacro:wheel_collision side="front_left"  />
+  <xacro:wheel_collision side="front_right"  />
+  <xacro:wheel_collision side="back_left" />
+  <xacro:wheel_collision side="back_right" />
   <!-- ROS 2 Control -->
   <gazebo>
