Commit message: Add rgbd camera

File: delivery_description/urdf/delivery_gazebo.xacro (robot description, xacro)
@@ -161,130 +161,30 @@
     </sensor>
   </gazebo>
-  <gazebo reference="camera_link">
-        <sensor name="camera" type="camera">
-            <camera>
-                <horizontal_fov>1.3962634</horizontal_fov>
-                <image>
-                    <width>640</width>
-                    <height>480</height>
-                    <format>R8G8B8</format>
-                </image>
-                <clip>
-                    <near>0.1</near>
-                    <far>15</far>
-                </clip>
-                <noise>
-                    <type>gaussian</type>
-                    <mean>0.0</mean>
-                    <stddev>0.007</stddev>
-                </noise>
-                <optical_frame_id>camera_link_optical</optical_frame_id>
-                <camera_info_topic>camera/camera_info</camera_info_topic>
-            </camera>
-            <always_on>1</always_on>
-            <update_rate>5.0</update_rate>
-            <visualize>true</visualize>
-            <topic>camera/image_raw</topic>
-        </sensor>
-    </gazebo>
-<!-- Ultrasonic Front Sensor -->
-<gazebo reference="ultrasonic_front_link">
-  <sensor name="ultrasonic_front" type="ray">
-    <always_on>true</always_on>
-    <update_rate>10</update_rate>
-    <visualize>true</visualize>
-    <topic>/ultrasonic/front</topic>
-    <gz_frame_id>ultrasonic_front_link</gz_frame_id>
-    <ray>
-      <scan>
-        <horizontal>
-          <samples>5</samples>
-          <resolution>1</resolution>
-          <min_angle>-0.05</min_angle>
-          <max_angle>0.05</max_angle>
-        </horizontal>
-      </scan>
-      <range>
-        <min>0.02</min>
-        <max>4.0</max>
-        <resolution>0.01</resolution>
-      </range>
-    </ray>
-  </sensor>
-</gazebo>
-<!-- Ultrasonic Back Sensor -->
-<gazebo reference="ultrasonic_back_link">
-  <sensor name="ultrasonic_back" type="ray">
-    <always_on>true</always_on>
-    <update_rate>10</update_rate>
-    <visualize>true</visualize>
-    <topic>/ultrasonic/back</topic>
-    <gz_frame_id>ultrasonic_back_link</gz_frame_id>
-    <ray>
-      <scan>
-        <horizontal>
-          <samples>5</samples>
-          <resolution>1</resolution>
-          <min_angle>-0.05</min_angle>
-          <max_angle>0.05</max_angle>
-        </horizontal>
-      </scan>
-      <range>
-        <min>0.02</min>
-        <max>4.0</max>
-        <resolution>0.01</resolution>
-      </range>
-    </ray>
-  </sensor>
-</gazebo>
-<!-- Ultrasonic Left Sensor -->
-<gazebo reference="ultrasonic_left_link">
-  <sensor name="ultrasonic_left" type="ray">
-    <always_on>true</always_on>
-    <update_rate>10</update_rate>
-    <visualize>true</visualize>
-    <topic>/ultrasonic/left</topic>
-    <gz_frame_id>ultrasonic_left_link</gz_frame_id>
-    <ray>
-      <scan>
-        <horizontal>
-          <samples>5</samples>
-          <resolution>1</resolution>
-          <min_angle>-0.05</min_angle>
-          <max_angle>0.05</max_angle>
-        </horizontal>
-      </scan>
-      <range>
-        <min>0.02</min>
-        <max>4.0</max>
-        <resolution>0.01</resolution>
-      </range>
-    </ray>
-  </sensor>
-</gazebo>
-<!-- Ultrasonic Right Sensor -->
-<gazebo reference="ultrasonic_right_link">
-  <sensor name="ultrasonic_right" type="ray">
-    <always_on>true</always_on>
-    <update_rate>10</update_rate>
-    <visualize>true</visualize>
-    <topic>/ultrasonic/right</topic>
-    <gz_frame_id>ultrasonic_right_link</gz_frame_id>
-    <ray>
-      <scan>
-        <horizontal>
-          <samples>5</samples>
-          <resolution>1</resolution>
-          <min_angle>-0.05</min_angle>
-          <max_angle>0.05</max_angle>
-        </horizontal>
-      </scan>
-      <range>
-        <min>0.02</min>
-        <max>4.0</max>
-        <resolution>0.01</resolution>
-      </range>
-    </ray>
-  </sensor>
-</gazebo>
+<gazebo reference="camera_color_optical_frame">
+    <sensor name="realsense_rgbd_camera" type="rgbd_camera">
+      <always_on>true</always_on>
+      <update_rate>30.0</update_rate>
+      <topic>/camera</topic>
+      <gz_frame_id>camera_depth_optical_frame</gz_frame_id>
+      <camera>
+          <horizontal_fov>1.39626</horizontal_fov>
+          <image>
+              <width>640</width>
+              <height>480</height>
+              <format>R8G8B8</format>
+          </image>
+          <clip>
+              <near>0.2</near>
+              <far>10.0</far>
+          </clip>
+          <distortion>
+              <k1>0.0</k1>
+              <k2>0.0</k2>
+              <p1>0.0</p1>
+              <p2>0.0</p2>
+              <k3>0.0</k3>
+          </distortion>
+      </camera>
+    </sensor>
+  </gazebo>
 </robot>

File: delivery_description/urdf/sensors/realsense_d435.xacro (robot description, xacro)
@@ -1,10 +1,10 @@
 <?xml version="1.0"?>
 <robot  xmlns:xacro="http://ros.org/wiki/xacro">
-  <xacro:arg name="use_nominal_extrinsics" default="false"/>
+  <xacro:arg name="use_nominal_extrinsics" default="true"/>
   <xacro:arg name="add_plug" default="false" />
   <xacro:arg name="use_mesh" default="true" />
   <xacro:include filename="$(find realsense2_description)/urdf/_d435.urdf.xacro" />
   <xacro:sensor_d435 parent="base_link" use_nominal_extrinsics="$(arg use_nominal_extrinsics)" add_plug="$(arg add_plug)" use_mesh="$(arg use_mesh)">
-    <origin xyz="0.25 0 0.05" rpy="0 0 0"/>
+    <origin xyz="0.3 0 0.20" rpy="0 0 0"/>
   </xacro:sensor_d435>
 </robot>
