Commit message: change ultrasonig pose

File: delivery_description/urdf/sensors/ultrasonics.xacro (robot description, xacro)
@@ -1,32 +1,104 @@
 <?xml version="1.0" ?>
-<robot  xmlns:xacro="http://ros.org/wiki/xacro">
-   <xacro:macro name="ultrasonics" params="side offset_x offset_y rotate_z">
-        <link name="${side}_ultrasonic_link">
-            <visual>
-                <geometry>
-                    <box size="0.01 0.03 0.01" />
-                </geometry>
-                <origin xyz="0 0 0" rpy="0 0 0" />
-            </visual>
-            <collision>
-                <geometry>
-                    <box size="0.01 0.03 0.01" />
-                </geometry>
-                <origin xyz="0.01 0.03 0.01" rpy="0 0 0" />
-            </collision>
-        </link>
-        <joint name="${side}_ultrasonic_joint" type="fixed">
-            <parent link="base_link" />
-            <child link="${side}_ultrasonic_link" />
-            <origin xyz="${offset_x} ${offset_y} -0.05" rpy="0 0 ${rotate_z}"/>
-        </joint>
-   </xacro:macro>
-   <xacro:ultrasonics side="ffl" offset_x="0.27" offset_y="0.18" rotate_z="0" />
-   <xacro:ultrasonics side="ffr" offset_x="0.27" offset_y="-0.18" rotate_z="0" />
-   <xacro:ultrasonics side="bbl" offset_x="-0.27" offset_y="0.18" rotate_z="0" />
-   <xacro:ultrasonics side="bbr" offset_x="-0.27" offset_y="-0.18" rotate_z="0" />
-   <xacro:ultrasonics side="sfl" offset_x="0.12" offset_y="0.22" rotate_z="${pi/2}" />
-   <xacro:ultrasonics side="sbl" offset_x="-0.12" offset_y="0.22" rotate_z="${pi/2}" />
-   <xacro:ultrasonics side="sfr" offset_x="0.12" offset_y="-0.22" rotate_z="${pi/2}" />
-   <xacro:ultrasonics side="sbr" offset_x="-0.12" offset_y="-0.22" rotate_z="${pi/2}" />
+<robot xmlns:xacro="http://ros.org/wiki/xacro">
+  <xacro:macro name="ultrasonics" params="side offset_x offset_y rotate_z">
+    <link name="${side}_ultrasonic_link">
+      <visual>
+        <geometry>
+          <box size="0.01 0.03 0.01"/>
+        </geometry>
+        <origin xyz="0 0 0" rpy="0 0 0"/>
+        <material name="">
+          <color rgba="0.0 0.0 1.0 1" />
+        </material>
+      </visual>
+      <collision>
+        <geometry>
+          <box size="0.01 0.03 0.01"/>
+        </geometry>
+        <origin xyz="0 0 0" rpy="0 0 0"/>
+      </collision>
+      <inertial>
+        <mass value="0.01"/>
+        <origin xyz="0 0 0" rpy="0 0 0"/>
+        <inertia
+          ixx="1e-6"
+          ixy="0.0"
+          ixz="0.0"
+          iyy="1e-6"
+          iyz="0.0"
+          izz="1e-6"/>
+      </inertial>
+    </link>
+    <joint name="${side}_ultrasonic_joint" type="fixed">
+      <parent link="base_link"/>
+      <child link="${side}_ultrasonic_link"/>
+      <origin xyz="${offset_x} ${offset_y} -0.05" rpy="0 0 ${rotate_z}"/>
+    </joint>
+    <gazebo reference="${side}_ultrasonic_link">
+      <sensor name="${side}_ultrasonic" type="gpu_lidar">
+        <always_on>true</always_on>
+        <visualize>false</visualize>
+        <topic>${side}/range</topic>
+        <update_rate>5.0</update_rate>
+        <gz_frame_id>${side}_ultrasonic_link</gz_frame_id>
+        <lidar>
+          <scan>
+            <horizontal>
+              <samples>10</samples>
+              <resolution>1</resolution>
+              <min_angle>-0.1309</min_angle>
+              <max_angle>0.1309</max_angle>
+            </horizontal>
+          </scan>
+          <range>
+            <min>0.02</min>
+            <max>4.0</max>
+            <resolution>0.02</resolution>
+          </range>
+<!--
+          <noise>
+            <type>gaussian</type>
+            <mean>0.0</mean>
+            <stddev>0.01</stddev>
+          </noise> -->
+        </lidar>
+      </sensor>
+    </gazebo>
+  </xacro:macro>
+  <!-- Front -->
+  <xacro:ultrasonics side="ffl"
+                     offset_x="0.27"
+                     offset_y="0.18"
+                     rotate_z="0"/>
+  <xacro:ultrasonics side="ffr"
+                     offset_x="0.27"
+                     offset_y="-0.18"
+                     rotate_z="0"/>
+  <!-- Rear -->
+  <xacro:ultrasonics side="bbl"
+                     offset_x="-0.27"
+                     offset_y="0.18"
+                     rotate_z="${pi}"/>
+  <xacro:ultrasonics side="bbr"
+                     offset_x="-0.27"
+                     offset_y="-0.18"
+                     rotate_z="${pi}"/>
+  <!-- Left Side -->
+  <xacro:ultrasonics side="sfl"
+                     offset_x="0.12"
+                     offset_y="0.22"
+                     rotate_z="${pi/2}"/>
+  <xacro:ultrasonics side="sbl"
+                     offset_x="-0.12"
+                     offset_y="0.22"
+                     rotate_z="${pi/2}"/>
+  <!-- Right Side -->
+  <xacro:ultrasonics side="sfr"
+                     offset_x="0.12"
+                     offset_y="-0.22"
+                     rotate_z="${-pi/2}"/>
+  <xacro:ultrasonics side="sbr"
+                     offset_x="-0.12"
+                     offset_y="-0.22"
+                     rotate_z="${-pi/2}"/>
 </robot>
